Commit message: added some stuff for sim

File: scout_description/urdf/scout_mini/scout_mini.urdf (robot description, URDF)
Before this commit: robot scout_mini, 7 links, 6 joints
Links:
- removed link base_footprint
- added link base_scan; collision cylinder ; visual mesh filename=package://scout_description/meshes/scout_mini/mini_wheel.dae
- link base_link: geometry collision mesh filename=package://scout_description/meshes/scout_mini/mini_base_lin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; visual mesh filename=package://scout_description/meshes/scout_mini/mini_base_lin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
- link front_left_wheel_link: mass 1 -> 3; geometry collision mesh filename=package://scout_description/meshes/scout_mini/mini_wheel.dae; visual mesh filename=package://scout_description/meshes/scout_mini/mini_wheel.dae
- link front_right_wheel_link: mass 1 -> 3; geometry collision mesh filename=package://scout_description/meshes/scout_mini/mini_wheel.dae; visual mesh filename=package://scout_description/meshes/scout_mini/mini_wheel.dae
- link inertial_link: mass 18 -> 60
- link rear_left_wheel_link: mass 1 -> 3; geometry collision mesh filename=package://scout_description/meshes/scout_mini/mini_wheel.dae; visual mesh filename=package://scout_description/meshes/scout_mini/mini_wheel.dae
- link rear_right_wheel_link: mass 1 -> 3; geometry collision mesh filename=package://scout_description/meshes/scout_mini/mini_wheel.dae; visual mesh filename=package://scout_description/meshes/scout_mini/mini_wheel.dae
Joints:
- removed joint base_footprint_joint
- added joint lidar_joint: type fixed, parent , child , axis 
- joint front_left_wheel: axis 0 -1 0 -> 0 0 -1; origin xyz=0.226 0.245 -0.0905 rpy=0 0 0 -> xyz=0.2319755 0.2082515 -0.100998 rpy=-1.57 0 0
- joint front_right_wheel: axis 0 -1 0 -> 0 0 -1; origin xyz=0.226 -0.245 -0.0905 rpy=3.14 0 0 -> xyz=0.2319755 -0.2082515 -0.099998 rpy=1.57 0 0
- joint rear_left_wheel: axis 0 -1 0 -> 0 0 -1; origin xyz=-0.226 0.245 -0.0905 rpy=0 0 0 -> xyz=-0.2319755 0.2082515 -0.100998 rpy=-1.57 0 0
- joint rear_right_wheel: axis 0 -1 0 -> 0 0 -1; origin xyz=-0.226 -0.245 -0.0905 rpy=3.14 0 0 -> xyz=-0.2319755 -0.2082515 -0.099998 rpy=1.57 0 0

Commit message: fixed up visuals

File: scout_description/urdf/scout_mini/scout_mini.urdf (robot description, URDF)
Before this commit: robot scout_mini, 7 links, 6 joints
Links:
- added link base_footprint
- link base_link: geometry collision box size=0.595 0.395 0.13; visual mesh filename=package://scout_description/meshes/scout_mini/mini_base_lin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
- link base_scan: mass None -> 0.01; geometry collision cylinder length=0.055 radius=0.0508; visual mesh filename=package://scout_description/meshes/scout_mini/lds.dae scale=0.001 0.001 0.001
- link front_left_wheel_link: mass 3 -> 1; geometry collision cylinder length=0.0852 radius=0.0875; visual mesh filename=package://scout_description/meshes/scout_mini/mini_wheel.dae
- link front_right_wheel_link: mass 3 -> 1; geometry collision cylinder length=0.0852 radius=0.0875; visual mesh filename=package://scout_description/meshes/scout_mini/mini_wheel.dae
- link inertial_link: mass 60 -> 18
- link rear_left_wheel_link: mass 3 -> 1; geometry collision cylinder length=0.0852 radius=0.0875; visual mesh filename=package://scout_description/meshes/scout_mini/mini_wheel.dae
- link rear_right_wheel_link: mass 3 -> 1; geometry collision cylinder length=0.0852 radius=0.0875; visual mesh filename=package://scout_description/meshes/scout_mini/mini_wheel.dae
Joints:
- added joint base_footprint_joint: type fixed, parent base_link, child base_footprint, origin xyz=0 0 -0.178 rpy=0 0 0
- joint front_left_wheel: axis 0 0 -1 -> 0 -1 0; origin xyz=0.2319755 0.2082515 -0.100998 rpy=-1.57 0 0 -> xyz=0.226 0.245 -0.0905 rpy=0 0 0
- joint front_right_wheel: axis 0 0 -1 -> 0 -1 0; origin xyz=0.2319755 -0.2082515 -0.099998 rpy=1.57 0 0 -> xyz=0.226 -0.245 -0.0905 rpy=3.14 0 0
- joint lidar_joint: axis  -> 0 0 -1; child  -> base_scan; parent  -> base_link
- joint rear_left_wheel: axis 0 0 -1 -> 0 -1 0; origin xyz=-0.2319755 0.2082515 -0.100998 rpy=-1.57 0 0 -> xyz=-0.226 0.245 -0.0905 rpy=0 0 0
- joint rear_right_wheel: axis 0 0 -1 -> 0 -1 0; origin xyz=-0.2319755 -0.2082515 -0.099998 rpy=1.57 0 0 -> xyz=-0.226 -0.245 -0.0905 rpy=3.14 0 0

Commit message: dont' know wjhy old model was owrking weird

File: scout_description/urdf/scout_mini/scout_mini.urdf (robot description, URDF)
Before this commit: robot scout_mini, 8 links, 7 joints
Links:
- removed link base_footprint
- removed link base_scan
- link base_link: geometry collision mesh filename=package://scout_description/meshes/scout_mini/scout_mini_ba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; visual mesh filename=package://scout_description/meshes/scout_mini/scout_mini_ba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
- link front_left_wheel_link: mass 1 -> 3; geometry collision mesh filename=package://scout_description/meshes/scout_mini/wheel.dae; visual mesh filename=package://scout_description/meshes/scout_mini/wheel.dae
- link front_right_wheel_link: mass 1 -> 3; geometry collision mesh filename=package://scout_description/meshes/scout_mini/wheel.dae; visual mesh filename=package://scout_description/meshes/scout_mini/wheel.dae
- link inertial_link: mass 18 -> 132.3898489950015
- link rear_left_wheel_link: mass 1 -> 3; geometry collision mesh filename=package://scout_description/meshes/scout_mini/wheel.dae; visual mesh filename=package://scout_description/meshes/scout_mini/wheel.dae
- link rear_right_wheel_link: mass 1 -> 3; geometry collision mesh filename=package://scout_description/meshes/scout_mini/wheel.dae; visual mesh filename=package://scout_description/meshes/scout_mini/wheel.dae
Joints:
- removed joint base_footprint_joint
- removed joint lidar_joint
- joint front_left_wheel: axis 0 -1 0 -> 0 0 -1; origin xyz=0.226 0.245 -0.0905 rpy=0 0 0 -> xyz=-0.1566278 0.2281768 -0.077 rpy=0 -1.57 0
- joint front_right_wheel: axis 0 -1 0 -> 0 0 -1; origin xyz=0.226 -0.245 -0.0905 rpy=3.14 0 0 -> xyz=0.1566278 0.2281768 -0.077 rpy=0 1.57 0
- joint rear_left_wheel: axis 0 -1 0 -> 0 0 -1; origin xyz=-0.226 0.245 -0.0905 rpy=0 0 0 -> xyz=-0.1566278 -0.2281768 -0.077 rpy=0 -1.57 0
- joint rear_right_wheel: axis 0 -1 0 -> 0 0 -1; origin xyz=-0.226 -0.245 -0.0905 rpy=3.14 0 0 -> xyz=0.1566278 -0.2281768 -0.077 rpy=0 1.57 0

File: scout_description/urdf/scout_mini/scout_mini.xacro (robot description, xacro)
@@ -3,43 +3,69 @@
     xmlns:xacro="http://ros.org/wiki/xacro">
     <xacro:arg name="robot_namespace" default="/" />
-    <xacro:include filename="$(find scout_description)/urdf/scout_mini/scout_mini_wheel.xacro" />
+    <xacro:arg name="urdf_extras" default="empty.urdf" />
+    <xacro:include filename="$(find scout_description)/urdf/scout_mini/scout_mini_wheel_1.xacro" />
+    <xacro:include filename="$(find scout_description)/urdf/scout_mini/scout_mini_wheel_2.xacro" />
+    <xacro:include filename="$(find scout_description)/urdf/scout_mini/scout_mini_wheel_3.xacro" />
+    <xacro:include filename="$(find scout_description)/urdf/scout_mini/scout_mini_wheel_4.xacro" />
     <!-- Variables -->
     <xacro:property name="M_PI" value="3.14159"/>
     <!-- Vehicle Geometries -->
-    <xacro:property name="base_x_size" value="0.595000" />
-    <!-- <xacro:property name="base_y_size" value="0.335000" /> -->
-    <xacro:property name="base_y_size" value="0.395000" />
-    <xacro:property name="base_z_size" value="0.130000" />
-    <xacro:property name="wheelbase" value="0.452" />
-    <xacro:property name="track" value="0.49" />
-    <xacro:property name="wheel_vertical_offset" value="-0.0905" />
-    <xacro:property name="wheel_length" value="0.8520e-01" />
-    <xacro:property name="wheel_radius" value="0.8750e-01" />
+    <xacro:property name="base_x_size" value="0.6200000" />
+    <xacro:property name="base_y_size" value="0.585000" />
+    <xacro:property name="base_z_size" value="0.235000" />
+    <xacro:property name="wheelbase" value="0.3132556"/>
+   <xacro:property name="track" value="0.4563536" />
+   <xacro:property name="wheel_vertical_offset" value="-0.077" />
+<!--    <xacro:property name="track" value="0.3426" />
+    <xacro:property name="wheelbase" value="0.3181"/>
+    <xacro:property name="wheel_vertical_offset" value="-0.160000047342231" />-->
+    <xacro:property name="wheel_length" value="0.8e-01" />
+    <xacro:property name="wheel_radius" value="1.600e-01" />
     <!-- Base link -->
     <link name="base_link">
         <visual>
-            <origin xyz="0 0 0" rpy="0 0 0" />
+            <!--origin xyz="-0.0145261552504705 0.0231316650320557 0.00586280190939592" rpy="0 0 0" /-->
+            <origin xyz="0.015 0.0231316650320557 0" rpy="0 0 0"/>
+            <!--<origin
+              xyz="-0.0145261552504705 0.0231316650320557 0.00586280190939592"
+              rpy="0 0 0" />-->
             <geometry>
-                <mesh filename="package://scout_description/meshes/scout_mini/mini_base_link.dae" />
+                <mesh filename="package://scout_description/meshes/scout_mini/scout_mini_base_link.STL" />
             </geometry>
         </visual>
         <collision>
-            <origin xyz="0 0 0.008" rpy="0 0 0" />
-            <geometry>
-                <box size="${base_x_size} ${base_y_size} ${base_z_size}"/>
-            </geometry>
+          <!--origin
+            xyz="-0.0145261552504705 0.0231316650320557 0.00586280190939592"
+            rpy="0 0 0" /-->
+            <origin xyz="0.015 0.0231316650320557 0" rpy="0 0 0"/>
+          <geometry>
+            <mesh
+              filename="package://scout_description/meshes/scout_mini/scout_mini_base_link.STL" />
+          </geometry>
         </collision>
     </link>
-    <link name="base_footprint"/>
-    <joint name="base_footprint_joint" type="fixed">
-        <origin xyz="0 0 ${wheel_vertical_offset - wheel_radius}" rpy="0 0 0" />
+    <!-- <joint name="chassis_link_joint" type="fixed">
+        <origin xyz="0 0 ${wheel_radius - wheel_vertical_offset}" rpy="0 0 0" />
         <parent link="base_link" />
-        <child link="base_footprint" />
-    </joint>
+        <child link="chassis_link" />
+    </joint> -->
     <link name="inertial_link">
         <inertial>
-            <mass value="18" />
-            <origin xyz="0.0 0.0 0.0" />
-            <inertia ixx="2.288641" ixy="0" ixz="0" iyy="5.103976" iyz="0" izz="3.431465" />
+            <!--mass value="44.3898489950015" /-->
+            <mass value="132.3898489950015" />
+            <!-- <mass value="50" /> -->
+            <!-- <origin xyz="-0.00065 -0.085 0.062" />
+            <inertia ixx="0.6022" ixy="-0.02364" ixz="-0.1197" iyy="1.7386" iyz="-0.001544" izz="2.0296" /> -->
+            <origin xyz="0.015 0.0231316650320557 0" />
+            <!--<origin
+              xyz="-0.0145261552504705 0.0231316650320557 0.00586280190939592"
+              rpy="0 0 0" />-->
+            <inertia ixx="0.185196122711036"
+            ixy="4.30144213829512E-08"
+            ixz="5.81037523686401E-08"
+            iyy="0.364893736238929"
+            iyz="-0.000386720198091934"
+            izz="0.223868521722778" />
+            <!--<inertia ixx="2.288641" ixy="0" ixz="0" iyy="5.103976" iyz="0" izz="3.431465" />-->
         </inertial>
     </link>
@@ -49,18 +75,29 @@
         <child link="inertial_link" />
     </joint>
+    <!-- For testing, hang the robot up in the air -->
+    <!-- <link name="world" />
+    <joint name="world_to_base_link=" type="fixed">
+        <origin xyz="0 0 0.5" rpy="0 0 0" />
+        <parent link="world"/>
+        <child link="base_link"/>
+    </joint> -->
     <!-- Scout wheel macros -->
     <!-- wheel labeled from 0 to 3, conter-clockwise, starting from front right wheel -->
     <!-- motor 1 and 2 (left side) are mechanically installed in a reversed direction -->
-    <xacro:scout_mini_wheel wheel_prefix="front_right">
-        <origin xyz="${wheelbase/2} ${-track/2} ${wheel_vertical_offset}" rpy="3.14 0 0" />
-    </xacro:scout_mini_wheel>
-    <xacro:scout_mini_wheel wheel_prefix="front_left">
-        <origin xyz="${wheelbase/2} ${track/2} ${wheel_vertical_offset}" rpy="0 0 0" />
-    </xacro:scout_mini_wheel>
-    <xacro:scout_mini_wheel wheel_prefix="rear_left">
-        <origin xyz="${-wheelbase/2} ${track/2} ${wheel_vertical_offset}" rpy="0 0 0" />
-    </xacro:scout_mini_wheel>
-    <xacro:scout_mini_wheel wheel_prefix="rear_right">
-        <origin xyz="${-wheelbase/2} ${-track/2} ${wheel_vertical_offset}" rpy="3.14 0 0" />
-    </xacro:scout_mini_wheel>
+    <xacro:scout_mini_wheel_1 wheel_prefix="rear_right">
+        <origin xyz="${wheelbase/2} ${-track/2} ${wheel_vertical_offset}" rpy="0 1.57 0" />
+    </xacro:scout_mini_wheel_1>
+    <xacro:scout_mini_wheel_2 wheel_prefix="front_right">
+        <origin xyz="${wheelbase/2} ${track/2} ${wheel_vertical_offset}" rpy="0 1.57 0" />
+    </xacro:scout_mini_wheel_2>
+    <xacro:scout_mini_wheel_3 wheel_prefix="front_left">
+        <origin xyz="${-wheelbase/2} ${track/2} ${wheel_vertical_offset}" rpy="0 -1.57 0" />
+    </xacro:scout_mini_wheel_3>
+    <xacro:scout_mini_wheel_4 wheel_prefix="rear_left">
+        <origin xyz="${-wheelbase/2} ${-track/2} ${wheel_vertical_offset}" rpy="0 -1.57 0" />
+    </xacro:scout_mini_wheel_4>
+    <!-- Additional definitions -->
+    <xacro:include filename="$(arg urdf_extras)" />
+    <!-- Gazebo definitions  -->
+    <xacro:include filename="$(find scout_description)/urdf/scout_mini/scout_mini.gazebo" />
 </robot>
