Commit message: Added lidar and depth cam functioinality

File: scout_description/urdf/grogu.xacro (robot description, xacro)
@@ -1,11 +1,11 @@
 <?xml version="1.0"?>
-<robot name="scout_mini"
+<robot name="grogu"
     xmlns:xacro="http://ros.org/wiki/xacro">
     <xacro:arg name="robot_namespace" default="/" />
     <xacro:arg name="urdf_extras" default="empty.urdf" />
-    <xacro:include filename="$(find scout_description)/urdf/scout_mini_wheel_1.xacro" />
-    <xacro:include filename="$(find scout_description)/urdf/scout_mini_wheel_2.xacro" />
-    <xacro:include filename="$(find scout_description)/urdf/scout_mini_wheel_3.xacro" />
-    <xacro:include filename="$(find scout_description)/urdf/scout_mini_wheel_4.xacro" />
+    <xacro:include filename="$(find scout_description)/urdf/grogu_wheel_1.xacro" />
+    <xacro:include filename="$(find scout_description)/urdf/grogu_wheel_2.xacro" />
+    <xacro:include filename="$(find scout_description)/urdf/grogu_wheel_3.xacro" />
+    <xacro:include filename="$(find scout_description)/urdf/grogu_wheel_4.xacro" />
     <!-- Variables -->
     <xacro:property name="M_PI" value="3.14159"/>
@@ -29,5 +29,5 @@
                     rpy="1.57 0 -1.57" />
             <geometry>
-                <mesh filename="package://scout_description/meshes/scout_mini_base_link2.dae" />
+                <mesh filename="file://$(find scout_description)/meshes/grogu_base_link2.dae" />
             </geometry>
         </visual>
@@ -37,12 +37,11 @@
                     rpy="1.57 0 -1.57" />
           <geometry>
-            <mesh
-              filename="package://scout_description/meshes/scout_mini_base_link2.dae" />
+            <mesh filename="file://$(find scout_description)/meshes/grogu_base_link2.dae" />
           </geometry>
         </collision>
     </link>
-    <link name="base_scan">
+    <link name="base_scan_lidar">
       <collision name="lidar_sensor_collision">
-        <origin xyz="-0.020 0 0.161" rpy="0 0 0"/>
+        <origin xyz="-0.020 0 -0.1" rpy="0 0 0"/>
         <geometry>
           <cylinder radius="0.0508" length="0.055"/>
@@ -50,5 +49,5 @@
       </collision>
       <visual name="lidar_sensor_visual">
-        <origin xyz="-0.032 0 0.171" rpy="0 0 0"/>
+        <origin xyz="-0.032 0 -0.1" rpy="0 0 0"/>
         <geometry>
           <cylinder radius="0.0508" length="0.055"/>
@@ -56,4 +55,20 @@
       </visual>
     </link>
+    <link name="base_scan_camera">
+      <collision name="camera_collision">
+        <origin xyz="0.01 0.0 0.0" rpy="0.0 0.0 0.0"/>
+        <geometry>
+          <cylinder radius="0.012" length="0.01"/>
+        </geometry>
+      </collision>
+      <visual name="camera_visual">
+        <origin xyz="0.01 0.0 0.0" rpy="0.0 ${pi/2} 0.0"/>
+        <geometry>
+          <cylinder radius="0.012" length="0.01"/>
+        </geometry>
+      </visual>
+    </link>
+    <!-- for conversion from ros coords to image -->
+    <link name="base_scan_camera_optical"></link>
     <!-- <joint name="chassis_link_joint" type="fixed">
         <origin xyz="0 0 ${wheel_radius - wheel_vertical_offset}" rpy="0 0 0" />
@@ -63,8 +78,14 @@
     <link name="inertial_link">
         <inertial>
-            <mass value="60" />
+            <mass value="36" />
             <origin xyz="0.0 0.0 0.0" />
             <inertia ixx="2.288641" ixy="0" ixz="0" iyy="5.103976" iyz="0" izz="3.431465" />
         </inertial>
+        <visual name="imu_visual">
+        <origin xyz="0.01 0.0 0.2" rpy="0.0 ${pi/2} 0.0"/>
+        <geometry>
+          <cylinder radius="0.012" length="0.01"/>
+        </geometry>
+      </visual>
     </link>
     <joint name="inertial_joint" type="fixed">
@@ -75,7 +96,17 @@
     <joint name="lidar_joint" type="fixed">
         <parent link="base_link"/>
-        <child link="base_scan"/>
+        <child link="base_scan_lidar"/>
         <origin xyz="-0.032 0 0.171" rpy="0 0 0"/>
-        <axis xyz="0 0 1" rpy="0 0 0"/>
+    </joint>
+    <joint name="camera_joint" type="fixed">
+        <parent link="base_link"/>
+        <child link="base_scan_camera"/>
+        <origin xyz="0.26 0.0 0.03" rpy="0.0 0.0 0.0"/>
+    </joint>
+    <!-- Translates between ros coords and image direction -->
+    <joint name="camera_optical_joint" type="fixed">
+        <parent link="base_scan_camera"/>
+        <child link="base_scan_camera_optical"/>
+        <origin xyz="0.26 0.0 0.03" rpy="${-pi/2} 0 ${-pi/2}"/>
     </joint>
     <!-- For testing, hang the robot up in the air -->
@@ -89,31 +120,31 @@
     <!-- wheel labeled from 0 to 3, conter-clockwise, starting from front right wheel -->
     <!-- motor 1 and 2 (left side) are mechanically installed in a reversed direction -->
-    <xacro:scout_mini_wheel_1 wheel_prefix="front_left">
+    <xacro:grogu_wheel_1 wheel_prefix="front_left">
     <!--<origin
             xyz="0 0 0"
             rpy="0 0 0" />-->
         <origin xyz="${wheelbase/2} ${track/2} ${wheel_vertical_offset}" rpy="-1.57 0 0" />
-    </xacro:scout_mini_wheel_1>
-    <xacro:scout_mini_wheel_2 wheel_prefix="rear_left">
+    </xacro:grogu_wheel_1>
+    <xacro:grogu_wheel_2 wheel_prefix="rear_left">
     <!--<origin
             xyz="0 0 0"
             rpy="0 0 0" />-->
         <origin xyz="${-wheelbase/2} ${track/2} ${wheel_vertical_offset}" rpy="-1.57 0 0" />
-    </xacro:scout_mini_wheel_2>
-    <xacro:scout_mini_wheel_3 wheel_prefix="front_right">
+    </xacro:grogu_wheel_2>
+    <xacro:grogu_wheel_3 wheel_prefix="front_right">
     <!--<origin
             xyz="0 0 0"
             rpy="0 0 0" />-->
         <origin xyz="${wheelbase/2} ${-track/2} ${wheel_vertical_offset+0.001}" rpy="1.57 0 0" />
-    </xacro:scout_mini_wheel_3>
-    <xacro:scout_mini_wheel_4 wheel_prefix="rear_right">
+    </xacro:grogu_wheel_3>
+    <xacro:grogu_wheel_4 wheel_prefix="rear_right">
     <!--<origin
            xyz="0 0 0"
            rpy="0 0 0" />-->
         <origin xyz="${-wheelbase/2} ${-track/2} ${wheel_vertical_offset+0.001}" rpy="1.57 0 0" />
-    </xacro:scout_mini_wheel_4>
+    </xacro:grogu_wheel_4>
     <!-- Additional definitions -->
     <xacro:include filename="$(arg urdf_extras)" />
     <!-- Gazebo definitions  -->
-    <xacro:include filename="$(find scout_description)/urdf/scout_mini.gazebo" />
+    <xacro:include filename="$(find scout_description)/urdf/grogu.gazebo" />
 </robot>

File: scout_description/urdf/grogu_wheel_1.xacro (robot description, xacro)
@@ -24,13 +24,13 @@
 -->
 <robot xmlns:xacro="http://ros.org/wiki/xacro" name="scout_wheel">
-    <xacro:macro name="scout_mini_wheel_2" params="wheel_prefix *joint_pose">
+    <xacro:macro name="grogu_wheel_1" params="wheel_prefix *joint_pose">
         <link name="${wheel_prefix}_wheel_link">
             <!--<inertial>
-            <mass value="3" />
+                <mass value="3" />
                 <origin
-                        xyz="0.162297526351148 0.159063056237198 -0.160000047342231"
+                        xyz="0.162297526351145 -0.159063056237197 -0.159999952657767"
                         rpy="0 0 0" />
                         <inertia ixx="0.7171" ixy="0" ixz="0" iyy="0.1361" iyz="0" izz="0.7171" />
-            </inertial>
+                   </inertial>
             <visual>
                 <origin xyz="0 0 0" rpy="0 0 0" />
@@ -63,6 +63,6 @@
         <joint name="${wheel_prefix}_wheel" type="continuous">
             <!--<origin
-                  xyz="-0.17453 0.20835 -0.07424"
-                  rpy="0 -1.57 0" />-->
+                  xyz="0.14547 0.20835 -0.07424"
+                  rpy="0 1.57 0" />-->
             <parent link="base_link"/>
             <child link="${wheel_prefix}_wheel_link"/>

File: scout_description/urdf/grogu_wheel_2.xacro (robot description, xacro)
@@ -24,31 +24,31 @@
 -->
 <robot xmlns:xacro="http://ros.org/wiki/xacro" name="scout_wheel">
-    <xacro:macro name="scout_mini_wheel_4" params="wheel_prefix *joint_pose">
+    <xacro:macro name="grogu_wheel_2" params="wheel_prefix *joint_pose">
         <link name="${wheel_prefix}_wheel_link">
-        <!--<inertial>
-        <mass value="3" />
-            <origin
-                    xyz="0.235244832119832 -0.0585653794466942 -0.206994929144493"
-                    rpy="0 0 0" />
-                    <inertia ixx="0.7171" ixy="0" ixz="0" iyy="0.1361" iyz="0" izz="0.7171" />
-        </inertial>
-        <visual>
-            <origin xyz="0 0 0" rpy="0 0 0" />
-            <geometry>
-                <mesh filename="package://scout_description/meshes/wheel.dae" />
-            </geometry>
-        </visual>-->
-        <inertial>
+            <!--<inertial>
             <mass value="3" />
-            <origin xyz="0 0 0" />
-            <inertia ixx="0.7171" ixy="0" ixz="0" iyy="0.7171" iyz="0" izz="0.1361" />
-            <!--<inertia ixx="0" ixy="0" ixz="0" iyy="0" iyz="0" izz="0" />-->
-        </inertial>
-        <visual>
-            <origin xyz="0 0 0" rpy="0 0 0" />
-            <geometry>
-                <mesh filename="package://scout_description/meshes/wheel.dae" />
-            </geometry>
-        </visual>
+                <origin
+                        xyz="0.162297526351148 0.159063056237198 -0.160000047342231"
+                        rpy="0 0 0" />
+                        <inertia ixx="0.7171" ixy="0" ixz="0" iyy="0.1361" iyz="0" izz="0.7171" />
+            </inertial>
+            <visual>
+                <origin xyz="0 0 0" rpy="0 0 0" />
+                <geometry>
+                    <mesh filename="package://scout_description/meshes/wheel.dae" />
+                </geometry>
+            </visual>-->
+            <inertial>
+                <mass value="3" />
+                <origin xyz="0 0 0" />
+                <inertia ixx="0.7171" ixy="0" ixz="0" iyy="0.7171" iyz="0" izz="0.1361" />
+                <!--<inertia ixx="0" ixy="0" ixz="0" iyy="0" iyz="0" izz="0" />-->
+            </inertial>
+            <visual>
+                <origin xyz="0 0 0" rpy="0 0 0" />
+                <geometry>
+                    <mesh filename="package://scout_description/meshes/wheel.dae" />
+                </geometry>
+            </visual>
             <collision>
               <origin
@@ -63,10 +63,10 @@
         <joint name="${wheel_prefix}_wheel" type="continuous">
             <!--<origin
-                  xyz="0.19247 -0.24486 -0.073441"
-                  rpy="-0 1.57 0" />-->
+                  xyz="-0.17453 0.20835 -0.07424"
+                  rpy="0 -1.57 0" />-->
             <parent link="base_link"/>
             <child link="${wheel_prefix}_wheel_link"/>
             <xacro:insert_block name="joint_pose"/>
-            <axis xyz="0 0 -1" rpy="0 0 0" />
+            <axis xyz="0 0 1" rpy="0 0 0" />
         </joint>
     </xacro:macro>

File: scout_description/urdf/grogu_wheel_3.xacro (robot description, xacro)
@@ -24,13 +24,13 @@
 -->
 <robot xmlns:xacro="http://ros.org/wiki/xacro" name="scout_wheel">
-    <xacro:macro name="scout_mini_wheel_1" params="wheel_prefix *joint_pose">
+    <xacro:macro name="grogu_wheel_3" params="wheel_prefix *joint_pose">
         <link name="${wheel_prefix}_wheel_link">
             <!--<inertial>
-                <mass value="3" />
+            <mass value="3" />
                 <origin
-                        xyz="0.162297526351145 -0.159063056237197 -0.159999952657767"
+                        xyz="-0.235088020493741 -0.0575697183039213 -0.16000004734223"
                         rpy="0 0 0" />
                         <inertia ixx="0.7171" ixy="0" ixz="0" iyy="0.1361" iyz="0" izz="0.7171" />
-                   </inertial>
+            </inertial>
             <visual>
                 <origin xyz="0 0 0" rpy="0 0 0" />
@@ -63,10 +63,10 @@
         <joint name="${wheel_prefix}_wheel" type="continuous">
             <!--<origin
-                  xyz="0.14547 0.20835 -0.07424"
-                  rpy="0 1.57 0" />-->
+                  xyz="-0.17453 -0.24424 -0.07424"
+                  rpy="0 -1.57 0" />-->
             <parent link="base_link"/>
             <child link="${wheel_prefix}_wheel_link"/>
             <xacro:insert_block name="joint_pose"/>
-            <axis xyz="0 0 1" rpy="0 0 0" />
+            <axis xyz="0 0 -1" rpy="0 0 0" />
         </joint>
     </xacro:macro>

File: scout_description/urdf/grogu_wheel_4.xacro (robot description, xacro)
@@ -24,31 +24,31 @@
 -->
 <robot xmlns:xacro="http://ros.org/wiki/xacro" name="scout_wheel">
-    <xacro:macro name="scout_mini_wheel_3" params="wheel_prefix *joint_pose">
+    <xacro:macro name="grogu_wheel_4" params="wheel_prefix *joint_pose">
         <link name="${wheel_prefix}_wheel_link">
-            <!--<inertial>
+        <!--<inertial>
+        <mass value="3" />
+            <origin
+                    xyz="0.235244832119832 -0.0585653794466942 -0.206994929144493"
+                    rpy="0 0 0" />
+                    <inertia ixx="0.7171" ixy="0" ixz="0" iyy="0.1361" iyz="0" izz="0.7171" />
+        </inertial>
+        <visual>
+            <origin xyz="0 0 0" rpy="0 0 0" />
+            <geometry>
+                <mesh filename="package://scout_description/meshes/wheel.dae" />
+            </geometry>
+        </visual>-->
+        <inertial>
             <mass value="3" />
-                <origin
-                        xyz="-0.235088020493741 -0.0575697183039213 -0.16000004734223"
-                        rpy="0 0 0" />
-                        <inertia ixx="0.7171" ixy="0" ixz="0" iyy="0.1361" iyz="0" izz="0.7171" />
-            </inertial>
-            <visual>
-                <origin xyz="0 0 0" rpy="0 0 0" />
-                <geometry>
-                    <mesh filename="package://scout_description/meshes/wheel.dae" />
-                </geometry>
-            </visual>-->
-            <inertial>
-                <mass value="3" />
-                <origin xyz="0 0 0" />
-                <inertia ixx="0.7171" ixy="0" ixz="0" iyy="0.7171" iyz="0" izz="0.1361" />
-                <!--<inertia ixx="0" ixy="0" ixz="0" iyy="0" iyz="0" izz="0" />-->
-            </inertial>
-            <visual>
-                <origin xyz="0 0 0" rpy="0 0 0" />
-                <geometry>
-                    <mesh filename="package://scout_description/meshes/wheel.dae" />
-                </geometry>
-            </visual>
+            <origin xyz="0 0 0" />
+            <inertia ixx="0.7171" ixy="0" ixz="0" iyy="0.7171" iyz="0" izz="0.1361" />
+            <!--<inertia ixx="0" ixy="0" ixz="0" iyy="0" iyz="0" izz="0" />-->
+        </inertial>
+        <visual>
+            <origin xyz="0 0 0" rpy="0 0 0" />
+            <geometry>
+                <mesh filename="package://scout_description/meshes/wheel.dae" />
+            </geometry>
+        </visual>
             <collision>
               <origin
@@ -63,6 +63,6 @@
         <joint name="${wheel_prefix}_wheel" type="continuous">
             <!--<origin
-                  xyz="-0.17453 -0.24424 -0.07424"
-                  rpy="0 -1.57 0" />-->
+                  xyz="0.19247 -0.24486 -0.073441"
+                  rpy="-0 1.57 0" />-->
             <parent link="base_link"/>
             <child link="${wheel_prefix}_wheel_link"/>
