Commit message: updated files to dynamically find meshes

File: scout_description/urdf/grogu.urdf (robot description, URDF)
Before this commit: robot grogu, 9 links, 8 joints
Links:
- link base_link: geometry collision mesh filename=package://scout_description/meshes/grogu_base_link2.dae; visual mesh filename=package://scout_description/meshes/grogu_base_link2.dae

File: scout_description/urdf/grogu.xacro (robot description, xacro)
@@ -29,5 +29,5 @@
                     rpy="1.57 0 -1.57" />
             <geometry>
-                <mesh filename="file://$(find scout_description)/meshes/grogu_base_link2.dae" />
+                <mesh filename="package://scout_description/meshes/grogu_base_link2.dae" />
             </geometry>
         </visual>
@@ -37,5 +37,5 @@
                     rpy="1.57 0 -1.57" />
           <geometry>
-            <mesh filename="file://$(find scout_description)/meshes/grogu_base_link2.dae" />
+            <mesh filename="package://scout_description/meshes/grogu_base_link2.dae" />
           </geometry>
         </collision>
